File: hardware/pcbs/controller2.brd (EAGLE design)
At the start: 30 x 16 mm, 50 parts, among them U1 ATMEGA328

Commit message: Add resistor and capacitor values to schematic.
Parts:
- C1, C3, C4: value (none) -> 100nF
- C2: value (none) -> 10uF
- R1, R2, R3: value 1k -> 10k
- moved R1 0.41 mm to (20.5, 12.2)
Routing:
- net GND: track 14.5 -> 29.2 mm, vias 9 -> 10
- net RESET: track 15.7 -> 14.6 mm
- net MOSI: track 21.8 -> 22.6 mm

Commit message: Add blank pin driver. New initialization sequence. Add new led driver classes.
Connections:
- net N$4 renamed RX
Changed lines of the file:
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@@
 <wire x1="9.125" y1="4.43210625" x2="9.125" y2="5.2" width="0.3048" layer="16"/>
 </signal>
-<signal name="N$4">
+<signal name="RX">
 <contactref element="U1" pad="30"/>
 <contactref element="TP18" pad="TP"/>

Commit message: Add VPROG pin to controller2.
Parts:
- U$6: device bookla:EVQPSD -> bookla:EVQPSG02K
- moved R4 3.21 mm to (14.2, 0.70), turned to 0 degrees
- moved U$6 0.80 mm to (25.2, 12.8)
- moved R5 0.60 mm to (13.9, 9.75)
- moved C3 0.50 mm to (14.2, 2.00)
- moved C4 0.40 mm to (14.2, 3.20)
- moved C1 0.30 mm to (14.2, 4.40)
Connections:
- new net VPRG: U$1.P6, U$3.P6, U1.14
- net BLANK: now also U1.11; no longer U1.10
- net XLAT: now also U1.10; no longer U1.9
Routing:
- net VPRG: track 0.00 -> 34.0 mm, vias 0 -> 2
- net VCC: track 21.0 -> 26.9 mm
- net GND: track 29.2 -> 34.5 mm
- net N$8: track 2.81 -> 6.75 mm
- net BLANK: track 22.7 -> 22.0 mm
- net XLAT: track 27.3 -> 26.6 mm
- net GSCLK: track 30.4 -> 29.8 mm
