File: hardware/pcbs/controller2.sch (EAGLE design)
At the start: 50 parts, among them U1 ATMEGA328

Commit message: Add resistor and capacitor values to schematic.
Parts:
- C1, C3, C4: value (none) -> 100nF
- C2: value (none) -> 10uF
- R1, R2, R3: value 1k -> 10k
Changed lines of the file:
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@@
 <part name="FRAME1" library="frames" deviceset="A4L-LOC" device=""/>
 <part name="GND1" library="supply1" deviceset="GND" device=""/>
-<part name="R1" library="rcl" deviceset="R-EU_" device="R0603" value="1k"/>
-<part name="C1" library="rcl" deviceset="C-EU" device="C0603"/>
+<part name="R1" library="rcl" deviceset="R-EU_" device="R0603" value="10k"/>
+<part name="C1" library="rcl" deviceset="C-EU" device="C0603" value="100nF"/>
 <part name="U$6" library="bookla" deviceset="SWITCH" device=""/>
-<part name="C2" library="rcl" deviceset="C-EU" device="C0805"/>
+<part name="C2" library="rcl" deviceset="C-EU" device="C0805" value="10uF"/>
 <part name="P+2" library="supply1" deviceset="VCC" device=""/>
-<part name="R2" library="rcl" deviceset="R-EU_" device="R0603" value="1k"/>
-<part name="R3" library="rcl" deviceset="R-EU_" device="R0603" value="1k"/>
+<part name="R2" library="rcl" deviceset="R-EU_" device="R0603" value="10k"/>
+<part name="R3" library="rcl" deviceset="R-EU_" device="R0603" value="10k"/>
 <part name="U$1" library="niklas" deviceset="TLC5940" device=""/>
 <part name="U1" library="thecustomgeek" deviceset="ATMEGA328" device=""/>
@@
 <attribute name="TP_SIGNAL_NAME" value=""/>
 </part>
-<part name="C3" library="rcl" deviceset="C-EU" device="C0603"/>
-<part name="C4" library="rcl" deviceset="C-EU" device="C0603"/>
+<part name="C3" library="rcl" deviceset="C-EU" device="C0603" value="100nF"/>
+<part name="C4" library="rcl" deviceset="C-EU" device="C0603" value="100nF"/>
 <part name="P+7" library="supply1" deviceset="VCC" device=""/>
 <part name="GND9" library="supply1" deviceset="GND" device=""/>

Commit message: Add blank pin driver. New initialization sequence. Add new led driver classes.
Connections:
- net N$4 renamed RX
Changed lines of the file:
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@@
 </segment>
 </net>
-<net name="N$4" class="0">
+<net name="RX" class="0">
 <segment>
 <pinref part="U1" gate="G$1" pin="PD0(RXD)"/>

Commit message: Add VPROG pin to controller2.
Connections:
- new net VPRG: U$1.VPRG, U$3.VPRG, U1.PB2(SS/OC1B)
- net BLANK: now also U1.PD7(AIN1); no longer U1.PD6(AIN0)
- net XLAT: now also U1.PD6(AIN0); no longer U1.PD5(T1)
Changed lines of the file:
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@@
+</segment>
+<segment>
+<pinref part="U$3" gate="G$1" pin="BLANK"/>
+<wire x1="116.84" y1="53.34" x2="119.38" y2="53.34" width="0.1524" layer="91"/>
+<label x="119.38" y="53.34" size="1.27" layer="95" xref="yes"/>
+</segment>
+<segment>
+<pinref part="U1" gate="G$1" pin="PD7(AIN1)"/>
+<wire x1="109.22" y1="109.22" x2="111.76" y2="109.22" width="0.1524" layer="91"/>
+<label x="111.76" y="109.22" size="1.27" layer="95" xref="yes"/>
+</segment>
+</net>
+<net name="XLAT" class="0">
+<segment>
+<pinref part="U$1" gate="G$1" pin="XLAT"/>
+<wire x1="58.42" y1="55.88" x2="60.96" y2="55.88" width="0.1524" layer="91"/>
+<label x="60.96" y="55.88" size="1.27" layer="95" xref="yes"/>
+</segment>
+<segment>
+<pinref part="U$3" gate="G$1" pin="XLAT"/>
+<wire x1="116.84" y1="55.88" x2="119.38" y2="55.88" width="0.1524" layer="91"/>
+<label x="119.38" y="55.88" size="1.27" layer="95" xref="yes"/>
 </segment>
 <segment>
@@
 <label x="111.76" y="111.76" size="1.27" layer="95" xref="yes"/>
 </segment>
-<segment>
-<pinref part="U$3" gate="G$1" pin="BLANK"/>
-<wire x1="116.84" y1="53.34" x2="119.38" y2="53.34" width="0.1524" layer="91"/>
-<label x="119.38" y="53.34" size="1.27" layer="95" xref="yes"/>
-</segment>
-</net>
-<net name="XLAT" class="0">
-<segment>
-<pinref part="U$1" gate="G$1" pin="XLAT"/>
-<wire x1="58.42" y1="55.88" x2="60.96" y2="55.88" width="0.1524" layer="91"/>
-<label x="60.96" y="55.88" size="1.27" layer="95" xref="yes"/>
-</segment>
-<segment>
-<pinref part="U1" gate="G$1" pin="PD5(T1)"/>
-<wire x1="109.22" y1="114.3" x2="111.76" y2="114.3" width="0.1524" layer="91"/>
-<label x="111.76" y="114.3" size="1.27" layer="95" xref="yes"/>
-</segment>
-<segment>
-<pinref part="U$3" gate="G$1" pin="XLAT"/>
-<wire x1="116.84" y1="55.88" x2="119.38" y2="55.88" width="0.1524" layer="91"/>
-<label x="119.38" y="55.88" size="1.27" layer="95" xref="yes"/>
-</segment>
 </net>
 <net name="N$8" class="0">
@@
 </segment>
 </net>
+<net name="VPRG" class="0">
+<segment>
+<pinref part="U$1" gate="G$1" pin="VPRG"/>
+<wire x1="58.42" y1="63.5" x2="60.96" y2="63.5" width="0.1524" layer="91"/>
+<label x="60.96" y="63.5" size="1.27" layer="95" xref="yes"/>
+</segment>
+<segment>
+<pinref part="U$3" gate="G$1" pin="VPRG"/>
+<wire x1="116.84" y1="63.5" x2="119.38" y2="63.5" width="0.1524" layer="91"/>
+<label x="119.38" y="63.5" size="1.27" layer="95" xref="yes"/>
+</segment>
+<segment>
+<pinref part="U1" gate="G$1" pin="PB2(SS/OC1B)"/>
+<wire x1="109.22" y1="99.06" x2="111.76" y2="99.06" width="0.1524" layer="91"/>
+<label x="111.76" y="99.06" size="1.27" layer="95" xref="yes"/>
+</segment>
+</net>
