File: hardware/pcbs/controller.sch (EAGLE design)
At the start: 47 parts, among them U1 ATMEGA328

Commit message: Remove first two pcb iterations and replace with the third working one.
Parts:
- removed C2: (no value), rcl:C-EUC0805
- removed R1: 1k, rcl:R-EU_R0603
- added U$5: CSRCE8, bookla:CSRCE8
- C1: value (none) -> 100nF
- R2, R3: value 1k -> 10k
Connections:
- net N$4 renamed RX
- new net VPRG: U$1.VPRG, U$3.VPRG, U1.PB2(SS/OC1B)
- new net XLAT1: U$5.1, U1.PB6(XTAL1/TOSC1)
- new net XLAT2: U$5.3, U1.PB7(XTAL2/TOSC2)
- net BLANK: now also U1.PD7(AIN1); no longer U1.PD6(AIN0)
- net GND: now also U$5.2; no longer C2.1
- net RESET: no longer R1.2
- net VCC: now also U$1.DCPRG, U$3.DCPRG; no longer C2.2, R1.1
- net XLAT: now also U1.PD6(AIN0); no longer U1.PD5(T1)
Other:
- moved on the sheet: C1, R4, R5
